Commit message: update kinect rviz setting

File: config/kinect_world.urdf (robot description, URDF)
Before this commit: robot kinect, 2 links, 1 joints
Joints:
- joint kinect_location: origin xyz=0.2159 0 0.8 rpy=0 0.0261799 0 -> xyz=0.0 0 1.5 rpy=0.0 0.5 -0.64

Commit message: object_tracking added

File: config/kinect_world.urdf (robot description, URDF)
Before this commit: robot kinect, 2 links, 1 joints
Joints:
- joint kinect_location: origin xyz=0.0 0 1.5 rpy=0.0 0.5 -0.64 -> xyz=0.0 0 1.0 rpy=0.0 0.0 -0.64

Commit message: context particles added

File: config/kinect_world.urdf (robot description, URDF)
Before this commit: robot kinect, 2 links, 1 joints
Joints:
- joint kinect_location: origin xyz=0.0 0 1.0 rpy=0.0 0.0 -0.64 -> xyz=0.0 0 1.0 rpy=0.0 0.2 -0.0
